File: GB-ICECART-GB/GB-ICECART-GB.kicad_pcb (KiCad board)
At the start: 2 copper layers, 51.4 x 61 mm, 7 parts, among them J1 Conn_02x16_Odd_Even, J2 DNF

Commit message: Add model of design
Parts:
- added C10: 2.2uF, Capacitor_SMD:C_0603_1608Metric, F.Cu at (208.3, 58.4)
- added C11: 2.2uF, Capacitor_SMD:C_0603_1608Metric, F.Cu at (205.7, 35.6)
- added C13: 100nF, Capacitor_SMD:C_0603_1608Metric, F.Cu at (190.5, 58.4)
- added C14: 0.1uF, Capacitor_SMD:C_0603_1608Metric, F.Cu at (198.1, 61.0)
- added J9: RB1-125B8G1A, Connector_RJ:RJ45_UDE_RB1-125B8G1A, F.Cu at (213.4, 29.7)
- added Q1: AO3401A, Package_TO_SOT_SMD:SOT-23, F.Cu at (193.0, 68.6)
- added U2: STM32F407ZGTx, Package_QFP:LQFP-144_20x20mm_P0.5mm, F.Cu at (184.4, 40.7)
- added U3: HT75xx-1-SOT89, Package_TO_SOT_SMD:SOT-89-3, F.Cu at (172.7, 68.6)
- renumbered C1 to C15, R1 to R15
Connections:
- net /VIN renamed VIN
- net GND renamed VSSA
