File: GB-ICECART-GB/GB-ICECART-GB.kicad_pcb (KiCad board)
At the start: 2 copper layers, 51.4 x 61 mm, 15 parts, among them J1 Conn_02x16_Odd_Even, J2 DNF, J9 RB1-125B8G1A, Q1 AO3401A, U2 STM32F407ZGTx, U3 HT75xx-1-SOT89

Commit message: Add schematic and pcb design images
Parts:
- removed J9: RB1-125B8G1A, Connector_RJ:RJ45_UDE_RB1-125B8G1A
- added BT1: Battery_Cell, Battery:BatteryHolder_Keystone_3002_1x2032, F.Cu at (49.8, 30.0)
- added C1: 15p, Capacitor_SMD:C_0603_1608Metric, F.Cu at (33.5, 58.4)
- added C12, C9: 100nF, Capacitor_SMD:C_0603_1608Metric, F.Cu at (33.5, 58.4)
- added C16: 1uF, Capacitor_SMD:C_0603_1608Metric, F.Cu at (36.1, 52.3)
- added C2: 15p, Capacitor_SMD:C_0603_1608Metric, F.Cu at (79.5, 52.8)
- added C3: 2.2uF, Capacitor_SMD:C_0603_1608Metric, F.Cu at (33.5, 58.4)
- added C4: 2.2uF, Capacitor_SMD:C_0603_1608Metric, F.Cu at (39.1, 66.0)
- added C5: 10, Capacitor_SMD:C_0603_1608Metric, F.Cu at (32.5, 72.1)
- added C6: 100nF, Capacitor_SMD:C_0603_1608Metric, F.Cu at (79.5, 68.8)
- added C7: 100nF, Capacitor_SMD:C_0603_1608Metric, F.Cu at (19.1, 51.8)
- added C8: 100nF, Capacitor_SMD:C_0603_1608Metric, F.Cu at (79.5, 58.8)
- added J3: AudioJack3, Connector_Audio:Jack_3.5mm_CUI_SJ1-3523N_Horizontal, F.Cu at (116.8, 35.8)
- added J4: Conn_02x08_Odd_Even, Connector_IDC:IDC-Header_2x08_P2.54mm_Vertical_SMD, F.Cu at (92.7, 35.8)
- added J5: Micro_SD_Card_Det, Connector_Card:microSD_HC_Hirose_DM3AT-SF-PEJM5, F.Cu at (119.4, 50.8)
- added L1: L, Inductor_SMD:L_6.3x6.3_H3, F.Cu at (110.5, 62.8)
- added LD1: Green, LED_SMD:LED_0603_1608Metric, F.Cu at (79.7, 45.7)
- added LD2: Orange, LED_SMD:LED_0603_1608Metric, F.Cu at (79.5, 48.8)
- added LD3: RED, LED_SMD:LED_0603_1608Metric, F.Cu at (79.8, 42.7)
- added LD4: Blue, LED_SMD:LED_0603_1608Metric, F.Cu at (33.5, 58.4)
- added Q2: AO3401A, Package_TO_SOT_SMD:SOT-23, F.Cu at (47.8, 83.3)
- added R1, R2: 5k1, Resistor_SMD:R_0603_1608Metric, F.Cu at (33.5, 58.4)
- added R10, R11, R14: 47K, Resistor_SMD:R_0603_1608Metric, F.Cu at (33.5, 58.4)
- added R12: 100K, Resistor_SMD:R_0603_1608Metric, F.Cu at (33.5, 58.4)
- added R13: 47K, Resistor_SMD:R_0603_1608Metric, F.Cu at (31.5, 49.8)
- added R16: 0, Resistor_SMD:R_0603_1608Metric, F.Cu at (79.5, 64.8)
- added R3: 20, Resistor_SMD:R_0603_1608Metric, F.Cu at (35.1, 46.7)
- added R4: 20, Resistor_SMD:R_0603_1608Metric, F.Cu at (31.2, 66.0)
- added R5, R6, R7, R8: 510, Resistor_SMD:R_0603_1608Metric, F.Cu at (33.5, 58.4)
- added R9: 10k, Resistor_SMD:R_0603_1608Metric, F.Cu at (33.5, 58.4)
- added SW1: SW_Push, Button_Switch_SMD:SW_SPST_B3U-1000P, F.Cu at (22.5, 42.2)
- added U1: STM32F407ZGTx, Package_QFP:LQFP-144_20x20mm_P0.5mm, B.Cu at (94.0, 56.4)
- added Y1: Crystal 8M, Crystal:Crystal_SMD_TXC_7M-4Pin_3.2x2.5mm, F.Cu at (48.3, 44.7)
- C10: value 2.2uF -> 100nF
- C11: value 2.2uF -> 0.1uF
- C14, C15: value 0.1uF -> 100nF
- D1: value LED_R -> D_Schottky; footprint LED_SMD:LED_0603_1608Metric -> Diode_SMD:D_0201_0603Metric
- J1: value Conn_02x16_Odd_Even -> DNF; footprint Connector_PinHeader_2.54mm:PinHeader_2x16_P2.54mm_Vertical_SMD -> Gekkio_Connector_PCBEdge:GameBoy_Cartridge_1x32_P1.50mm_Edge
- J2: value DNF -> TYPE-C-31-M-12; footprint Gekkio_Connector_PCBEdge:GameBoy_Cartridge_1x32_P1.50mm_Edge -> Connector_USB:USB_C_Receptacle_HRO_TYPE-C-31-M-12
- R15: value 3.3k -> 47K
- U2: value STM32F407ZGTx -> HT75xx-1-SOT89; footprint Package_QFP:LQFP-144_20x20mm_P0.5mm -> Package_TO_SOT_SMD:SOT-89-3
- U3: value HT75xx-1-SOT89 -> IS66WVS4M8BLL-104NLI; footprint Package_TO_SOT_SMD:SOT-89-3 -> IS66WVS4M8BLL:SOIC127P600X175-8N
- moved C10 174.8 mm to (33.5, 58.4)
- moved C11 173.7 mm to (33.5, 58.4)
- moved U2 166.5 mm to (19.9, 66.0)
- moved C13 161.1 mm to (29.5, 63.0)
- moved C14 150.2 mm to (48.3, 70.6)
- moved Q1 83.5 mm to (109.5, 70.8)
- moved U3 83.2 mm to (89.7, 74.5), turned to 180 degrees
- moved C15 49.8 mm to (125.5, 40.8)
- moved R15 44.2 mm to (114.5, 69.8)
- moved MK2 40.3 mm to (76.5, 26.8)
- moved J2 38.7 mm to (123.2, 65.0), turned to 90 degrees
- moved J1 36.9 mm to (102.6, 84.8), turned to 0 degrees
- moved D1 20.2 mm to (80.5, 61.8)
- moved MK1 11.5 mm to (102.5, 73.5)
Connections:
- C10 pad 1: Net-(C10-Pad1) -> VDD
- C11 pad 1: Net-(C11-Pad1) -> VSSA
- C11 pad 2: VSSA -> Net-(C11-Pad2)
- C13 pad 1: 3.3V -> VDD
- C14 pad 1: VSSA -> VDD
- C14 pad 2: Net-(C14-Pad2) -> VSSA
- C15 pad 1: +5V -> VDD
- D1 pad 1: VSSA -> VBAT
- D1 pad 2: Net-(D1-Pad2) -> Net-(BT1-Pad1)
- J1 pad 1: /A0 -> GB-VCC
- J1 pad 10: /~{CS} -> GB-A4
- J1 pad 11: /A5 -> GB-A5
- J1 pad 12: /D0 -> GB-A6
- J1 pad 13: /A6 -> GB-A7
- J1 pad 14: /D1 -> GB-A8
- J1 pad 15: /A7 -> GB-A9
- J1 pad 16: /D2 -> GB-A10
- J1 pad 17: /A8 -> GB-A11
- J1 pad 18: /D3 -> GB-A12
- J1 pad 19: /A9 -> GB-A13
- J1 pad 2: +5V -> GB-PHI
- J1 pad 20: /D4 -> GB-A14
- J1 pad 21: /A10 -> GB-A15
- J1 pad 22: /D5 -> GB-D0
- J1 pad 23: /A11 -> GB-D1
- J1 pad 24: /D6 -> GB-D2
- J1 pad 25: /A12 -> GB-D3
- J1 pad 26: /D7 -> GB-D4
- J1 pad 27: /A13 -> GB-D5
- J1 pad 28: /~{RES} -> GB-D6
- J1 pad 29: /A14 -> GB-D7
- J1 pad 3: /A1 -> GB-WR
- J1 pad 30: VIN -> GB-RES
- J1 pad 31: /A15 -> ADC-MIC2
- J1 pad 4: /PHI -> GB-RD
- J1 pad 5: /A2 -> GB-CS
- J1 pad 6: /~{WR} -> GB-A0
- J1 pad 7: /A3 -> GB-A1
- J1 pad 8: /~{RD} -> GB-A2
- J1 pad 9: /A4 -> GB-A3
- Q1 pad 3: Net-(C14-Pad2) -> Net-(C11-Pad2)
- R15 pad 1: +5V -> Net-(C11-Pad2)
- R15 pad 2: Net-(D1-Pad2) -> SD-D2
- U2 pad 1: unconnected-(U2-Pad1) -> VSSA
- U2 pad 2: unconnected-(U2-Pad2) -> GB-VCC
- U2 pad 3: unconnected-(U2-Pad3) -> 3.3V
- U3 pad 1: VSSA -> Mem_CS
- U3 pad 2: VIN -> Mem_SO
- U3 pad 3: 3.3V -> VSSA
Routing:
- net /D0: track 58.4 -> 0.00 mm, vias 3 -> 0
- net /D1: track 57.5 -> 0.00 mm, vias 3 -> 0
- net /D2: track 56.6 -> 0.00 mm, vias 3 -> 0
- net /D3: track 55.9 -> 0.00 mm, vias 3 -> 0
- net /D4: track 54.6 -> 0.00 mm, vias 1 -> 0
- net /~{RD}: track 54.6 -> 0.00 mm, vias 3 -> 0
- net /~{CS}: track 54.4 -> 0.00 mm, vias 3 -> 0
- net /D5: track 54.2 -> 0.00 mm, vias 1 -> 0
- net /~{WR}: track 54.1 -> 0.00 mm, vias 3 -> 0
- net /D6: track 53.7 -> 0.00 mm, vias 1 -> 0
- net /PHI: track 53.5 -> 0.00 mm, vias 3 -> 0
- net /D7: track 53.3 -> 0.00 mm, vias 1 -> 0
- net /~{RES}: track 52.9 -> 0.00 mm, vias 2 -> 0
- net VIN: track 52.4 -> 0.00 mm, vias 1 -> 0
- net /A15: track 50.7 -> 0.00 mm, vias 3 -> 0
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- added copper zone on F.Cu, net VDD
- removed copper zone on F.Cu, net +5V
