File: GB-ICECART-GB/GB-ICECART-GB.kicad_sch (KiCad schematic)
At the start: 46 parts, among them J1 Conn_02x16_Odd_Even, J2 DNF

Commit message: Add model of design
Parts:
- removed J1: Conn_02x16_Odd_Even, Connector_PinHeader_2.54mm:PinHeader_2x16_P2.54mm_Vertical_SMD, symbol Connector_Generic:Conn_02x16_Odd_Even
- removed J2: DNF, Gekkio_Connector_PCBEdge:GameBoy_Cartridge_1x32_P1.50mm_Edge, symbol Gekkio_Connector_Specialized:GameBoy_Cartridge
- added C12: 10, Capacitor_SMD:C_0603_1608Metric, symbol Device:C
- added J6: USB_B_Mini, Connector_USB:USB_Mini-B_Lumberg_2486_01_Horizontal, symbol Connector:USB_B_Mini
- added L1: L, Inductor_SMD:L_6.3x6.3_H3, symbol Device:L
- added R5, R7, R8: 20, Resistor_SMD:R_0603_1608Metric, symbol Device:R_US
- added R6: 11K, Resistor_SMD:R_0603_1608Metric, symbol Device:R_US
- C1, C2, C3, C4, C5, C6, C7, C8, C9: footprint (none) -> Capacitor_SMD:C_0603_1608Metric
- R1, R2, R3, R4: footprint (none) -> Resistor_SMD:R_0603_1608Metric
- R10, R11, R12, R13, R14, R9: renamed from R?; footprint (none) -> Resistor_SMD:R_0603_1608Metric
- gave numbers to parts that had none: 16
- renumbered C1 to C15, R1 to R15
Connections:
- net +5V: now also P1.A4 (VBUS), P1.A9 (VBUS), P1.B4 (VBUS), P1.B9 (VBUS), J6.1 (VBUS), R6.2
- net GND: now also P1.A1 (GND), P1.A12 (GND), P1.B1 (GND), P1.B12 (GND), P1.S1 (SHIELD), C12.1, J6.5 (GND), J6.6 (Shield)
- net USB_DM: now also R5.2, R6.1; no longer P1.A7 (D-)
- net USB_DP: now also R7.1; no longer P1.A6 (D+)
- net VDD: now also L1.2
- net USB_ID: now reaches U2.102 (PA10)
- net USB_ID: now also R8.1
- net VDDA: now reaches U2.32 (VREF+)
- net VDDA: now also C12.2, L1.1
- new net: J6.2 (D-), R7.2
- new net: J6.4 (ID), R8.2
- new net: J6.3 (D+), R5.1
Other:
- moved on the sheet: C10, C11, P1

Commit message: Update schematic and hook more up
Parts:
- removed C15: 0.1uF, Capacitor_SMD:C_0603_1608Metric, symbol Device:C
- removed D1: LED_R, LED_SMD:LED_0603_1608Metric, symbol Device:LED
- removed J5: AudioJack3, symbol Connector:AudioJack3
- removed J8: Conn_02x03_Odd_Even, symbol Connector_Generic:Conn_02x03_Odd_Even
- removed J9: RB1-125B8G1A, Connector_RJ:RJ45_UDE_RB1-125B8G1A, symbol Connector:RB1-125B8G1A
- removed P1: USB_C_Plug_USB2.0, symbol Connector:USB_C_Plug_USB2.0
- removed R15: 3.3k, Resistor_SMD:R_0603_1608Metric, symbol Device:R
- removed U1: IS66WVS4M8BLL-104NLI, symbol IS66WVS4M8BLL:IS66WVS4M8BLL-104NLI
- added BT1: Battery_Cell, symbol Device:Battery_Cell
- added C1, C2: 15p, Capacitor_SMD:C_0603_1608Metric, symbol Device:C
- added D1: D_Schottky, symbol Device:D_Schottky
- added Q2: AO3401A, Package_TO_SOT_SMD:SOT-23, symbol Transistor_FET:AO3401A
- added R12: 100K, Resistor_SMD:R_0603_1608Metric, symbol Device:R_US
- added R9: 10k, Resistor_SMD:R_0603_1608Metric, symbol Device:R_US
- added SW1: SW_Push, symbol Switch:SW_Push
- added U3: IS66WVS4M8BLL-104NLI, symbol IS66WVS4M8BLL:IS66WVS4M8BLL-104NLI
- added Y1: Crystal 8M, symbol Device:Crystal
- renumbered C4 to C10, C14 to C11, C5 to C12, C6 to C13, C7 to C14, C8 to C15, C9 to C16, C10 to C3, C11 to C4, C12 to C5, C1 to C6, C2 to C7, C3 to C8, C13 to C9, J6 to J1, J3 to J2, J4 to J3, J7 to J4, J10 to J6, R5 to R1, R9 to R10, R10 to R11, R11 to R13, R12 to R14, R13 to R15, R14 to R16, R6 to R2, R7 to R3, R8 to R4, R1 to R5, R2 to R6, R3 to R7, R4 to R8, U2 to U1, U3 to U2
Connections:
- net +5V is gone; now on net GB-VCC: J1.1 (VBUS), R2.2
- net GB-VIN is gone; now on net DAC-OUT2: J2.31 (VIN)
- net VIN is gone; now on net GB-VCC: U2.2 (VIN)
- net 3.3V: now also SW1.1, U3.8 (VDD)
- net GB-CS: now also U1.21 (PF9)
- net GB-PHI: now also U1.18 (PF6)
- net GB-RD: now also U1.20 (PF8)
- net GB-RES: now also U1.22 (PF10)
- net GB-VCC: now also Q2.1 (G), R12.1
- net GB-WR: now also U1.19 (PF7)
- net GND: now also C5.2, BT1.2 (-), C1.2, C2.2, R12.2, R9.2, U3.3 (SIO2), U3.4 (VSS), U3.7 (SIO3); no longer C5.1
- net SD-DET: now also U1.110 (PA15)
- net SD-ON: now also U1.109 (PA14)
- net VDD: now also L1.1; no longer L1.2
- net VDDA: now also C5.1, L1.2, U1.33 (VDDA); no longer C5.2, L1.1
- net GPIO0: now reaches J4.1 (Pin_1)
- net GPIO0: now also U1.56 (PG0)
- net GPIO9: now reaches J4.10 (Pin_10)
- net GPIO9: now also U1.124 (PG9)
- net GPIO10: now reaches J4.11 (Pin_11)
- net GPIO10: now also U1.125 (PG10)
- net GPIO11: now reaches J4.12 (Pin_12)
- net GPIO11: now also U1.126 (PG11)
- net GPIO12: now reaches J4.13 (Pin_13)
- net GPIO12: now also U1.127 (PG12)
- net GPIO13: now reaches J4.14 (Pin_14)
- net GPIO13: now also U1.128 (PG13)
- net GPIO14: now reaches J4.15 (Pin_15)
- net GPIO14: now also U1.129 (PG14)
- net GPIO15: now reaches J4.16 (Pin_16)
- net GPIO15: now also U1.132 (PG15)
- net GPIO1: now reaches J4.2 (Pin_2)
- net GPIO1: now also U1.57 (PG1)
- net GPIO2: now reaches J4.3 (Pin_3)
- net GPIO2: now also U1.87 (PG2)
- net GPIO3: now reaches J4.4 (Pin_4)
- net GPIO3: now also U1.88 (PG3)
- net GPIO4: now reaches J4.5 (Pin_5)
- net GPIO4: now also U1.89 (PG4)
- net GPIO5: now reaches J4.6 (Pin_6)
- net GPIO5: now also U1.90 (PG5)
- net GPIO6: now reaches J4.7 (Pin_7)
- net GPIO6: now also U1.91 (PG6)
- net GPIO7: now reaches J4.8 (Pin_8)
- net GPIO7: now also U1.92 (PG7)
- net GPIO8: now reaches J4.9 (Pin_9)
- net GPIO8: now also U1.93 (PG8)
- net LED1: now reaches U1.1 (PE2)
- net LED1: now also R6.1
- net Mem CLK: now reaches U1.133 (PB3)
- net Mem CLK: now also U3.6 (CLK)
- net Mem_SO: now reaches U1.134 (PB4)
- net Mem_SO: now also U3.2 (SO/SIO1)
- net Mem_SI: now reaches U1.135 (PB5)
- net Mem_SI: now also U3.5 (SI/SIO0)
- net Mem_CS: now reaches U1.136 (PB6)
- net Mem_CS: now also U3.1 (CE#)
- net at U1.138 (BOOT0): now also R9.1, SW1.2
- net LED2: now reaches U1.2 (PE3)
- net LED2: now also R7.1
- net at U1.23 (PH0): now also C1.1, Y1.1
- net at U1.24 (PH1): now also C2.1, Y1.2
- net LED3: now reaches U1.3 (PE4)
- net LED3: now also R8.1
- net DAC-OUT1: now reaches U1.40 (PA4)
- net DAC-OUT2: now reaches U1.41 (PA5)
- removed net PD?: R5.1, R6.1, R7.1, R8.1
- new net: BT1.1 (+), D1.2 (A), Q2.3 (D)
- new net PWR_LED: R5.1
- new net VCC: D1.1 (K), Q2.2 (S)
Other:
- note added: "Battery"
- note added: "Status LEDs"
- note removed: "Optional"
- company: https://gekkio.fi -> Iceberg Tech LLC.
- title: GB-BRK-CART -> GB-ICECART-GB
- moved on the sheet: C10, C11, C12, C13, C14, C15, C16, C3, C4, C5, C6, C7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

Commit message: Add schematic and pcb design images
Parts:
- removed J1: USB_B_Mini, Connector_USB:USB_Mini-B_Lumberg_2486_01_Horizontal, symbol Connector:USB_B_Mini
- removed R1: 20, Resistor_SMD:R_0603_1608Metric, symbol Device:R_US
- removed R2: 11K, Resistor_SMD:R_0603_1608Metric, symbol Device:R_US
- added J2: TYPE-C-31-M-12, Connector_USB:USB_C_Receptacle_HRO_TYPE-C-31-M-12, symbol Connector:USB_C_Receptacle_USB2.0
- added R1, R2: 5k1, Resistor_SMD:R_0603_1608Metric, symbol Device:R
- BT1: footprint (none) -> Battery:BatteryHolder_Keystone_3002_1x2032
- D1: footprint (none) -> Diode_SMD:D_0201_0603Metric
- J3: footprint (none) -> Connector_Audio:Jack_3.5mm_CUI_SJ1-3523N_Horizontal
- J4: footprint (none) -> Connector_IDC:IDC-Header_2x08_P2.54mm_Vertical_SMD
- J5: renamed from J6; footprint (none) -> Connector_Card:microSD_HC_Hirose_DM3AT-SF-PEJM5
- LD1, LD2, LD3, LD4: footprint (none) -> LED_SMD:LED_0603_1608Metric
- SW1: footprint (none) -> Button_Switch_SMD:SW_SPST_B3U-1000P
- U3: footprint (none) -> IS66WVS4M8BLL:SOIC127P600X175-8N
- Y1: footprint (none) -> Crystal:Crystal_SMD_TXC_7M-4Pin_3.2x2.5mm
- renumbered J2 to J1
Connections:
- net DAC-OUT1 is gone; now on net ADC-MIC1: U1.40 (PA4)
- net DAC-OUT2 is gone; now on net ADC-MIC2: J1.31 (VIN), U1.41 (PA5)
- net GB-VCC: now also J2.A4 (VBUS), J2.A9 (VBUS), J2.B4 (VBUS), J2.B9 (VBUS)
- net GND: now also J3.S, J5.11 (SHIELD), J2.A1 (GND), J2.A12 (GND), J2.B1 (GND), J2.B12 (GND), R1.2, R2.2
- net USB_DM: now also R4.2
- net USB_DP: now also R3.2; no longer R3.1
- net USB_ID: no longer R4.1
- net VBAT: now also D1.1 (K)
- net VDD: now also Q2.2 (S)
- net ADC-MIC2: now reaches J3.R
- net ADC-MIC2: now also U1.43 (PA7)
- net ADC-MIC1: now reaches J3.T
- net ADC-MIC1: now also U1.42 (PA6)
- removed net VCC: D1.1 (K), Q2.2 (S)
- new net: J2.A5 (CC1), R2.1
- new net: J2.A7 (D-), J2.B7 (D-), R3.1
- new net: J2.A6 (D+), J2.B6 (D+), R4.1
- new net: J2.B5 (CC2), R1.1
- new net SH: J2.S1 (SHIELD)
- no-connect marks 0 -> 3
Other:
- note added: "32Mbit Memory"
- note added: "Add way to switch between usb modes"
- note added: "Audio In/Out"
- note added: "Connectors"
- note added: "Gameboy Cartridge Pins"
- note added: "In operation, run midi keyboard from usb"
- note added: "In programing, program system from usb"
- note added: "Power Management"
- note added: "R: Ring / R"
- note added: "S: Sleeve / GND"
- note added: "SD Card"
- note added: "T: Tip / Left"
- note added: "USB Programming Port"
- note added: "Voltage regulator 5v -> 3.3v"
- title: GB-ICECART-GB -> ICECART-GB
- moved on the sheet: C5, J3, L1
