File: GB-ICECART-GB-Alpha/GB-ICECART-GB.kicad_pcb (KiCad board)
At the start: 2 copper layers, 51.4 x 61 mm, 53 parts, among them J1 DNF, J2 TYPE-C-31-M-12, J3 AudioJack3, J4 Conn_02x08_Odd_Even, J5 Micro_SD_Card_Det, Q1 AO3401A, Q2 AO3401A, SW1 SW_Push, U1 STM32F407ZGTx, U2 HT75xx-1-SOT89, U3 IS66WVS4M8BLL-104NLI, Y1 Crystal 8M

Commit message: Preliminary routing and BOM
Parts:
- removed BT1: Battery_Cell, Battery:BatteryHolder_Keystone_3002_1x2032
- removed D1: D_Schottky, Diode_SMD:D_0201_0603Metric
- removed MK2: DNF, Gekkio_MountingHole:MountingHole_2.3mm
- removed Q2: AO3401A, Package_TO_SOT_SMD:SOT-23
- removed R12: 100K, Resistor_SMD:R_0603_1608Metric
- U1: moved to F.Cu
- moved SW1 103.5 mm to (125.7, 33.8), turned to -90 degrees
- moved R9 94.2 mm to (125.9, 39.9)
- moved C10 91.2 mm to (122.7, 77.8)
- moved C5 90.2 mm to (122.7, 72.1)
- moved C7 83.5 mm to (102.1, 43.5), turned to 0 degrees
- moved R4 83.4 mm to (114.5, 63.6), turned to 180 degrees
- moved R1 82.8 mm to (116.3, 61.9), turned to 180 degrees
- moved C11 82.8 mm to (116.3, 60.3), turned to 180 degrees
- moved R2 82.7 mm to (115.5, 69.2)
- moved R3 81.9 mm to (114.5, 66.4), turned to 180 degrees
- moved R13 81.0 mm to (111.5, 62.5)
- moved R11 80.5 mm to (114.0, 60.2), turned to 90 degrees
- moved R14 79.8 mm to (111.5, 41.5)
- moved R10 78.9 mm to (112.4, 60.2), turned to 90 degrees
- moved LD4 78.6 mm to (108.9, 36.1), turned to 180 degrees
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Connections:
- net /SH renamed /SH_2
- C16 pad 1: VBAT -> Net-(C16-Pad1)
- LD1 pad 2: Net-(LD1-Pad2) -> Net-(LD1-A)
- LD2 pad 2: Net-(LD2-Pad2) -> Net-(LD2-A)
- LD3 pad 2: Net-(LD3-Pad2) -> Net-(LD3-A)
- R16 pad 2: VBAT -> Net-(C16-Pad1)
- R5 pad 1: PWR_LED -> VDD
- R5 pad 2: Net-(LD1-Pad2) -> Net-(LD2-A)
- R6 pad 2: Net-(LD2-Pad2) -> Net-(LD3-A)
- R7 pad 2: Net-(LD3-Pad2) -> Net-(LD1-A)
- SW1 pad 1: 3.3V -> VDD
- U1 pad 1: LED1 -> unconnected-(U1-PE2-Pad1)
- U1 pad 2: LED2 -> unconnected-(U1-PE3-Pad2)
- U1 pad 3: LED3 -> unconnected-(U1-PE4-Pad3)
- U1 pad 34: unconnected-(U1-Pad34) -> LED1
- U1 pad 35: unconnected-(U1-Pad35) -> LED2
- U1 pad 36: unconnected-(U1-Pad36) -> LED3
- U1 pad 6: VBAT -> unconnected-(U1-VBAT-Pad6)
Routing:
- net VDD: track 0.00 -> 201.5 mm, vias 0 -> 21
- net VSSA: track 5.45 -> 162.1 mm, vias 12 -> 20
- net ADC-MIC2: track 0.00 -> 76.2 mm, vias 0 -> 6
- net GB-VCC: track 0.00 -> 69.6 mm, vias 0 -> 2
- net GB-D7: track 0.00 -> 55.4 mm, vias 0 -> 2
- net GB-A15: track 0.00 -> 53.4 mm, vias 0 -> 2
- net GB-D6: track 0.00 -> 52.7 mm, vias 0 -> 2
- net SD-CMD: track 0.00 -> 52.6 mm, vias 0 -> 4
- net Net-(U1-BOOT0): track 0.00 -> 51.3 mm, vias 0 -> 2
- net GB-A14: track 2.63 -> 52.4 mm, vias 0 -> 2
- net GB-A13: track 2.25 -> 51.5 mm, vias 0 -> 2
- net SD-D0: track 0.00 -> 44.5 mm, vias 0 -> 3
- net SD-D1: track 0.00 -> 44.2 mm, vias 0 -> 3
- net SD-D3: track 0.00 -> 44.2 mm, vias 0 -> 2
- net GB-RES: track 0.00 -> 43.7 mm, vias 0 -> 2
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Other:
- board text removed: "+5V"
- board text removed: "A0"
- board text removed: "A1"
- board text removed: "A10"
- board text removed: "A11"
- board text removed: "A12"
- board text removed: "A13"
- board text removed: "A14"
- board text removed: "A15"
- board text removed: "A2"
- board text removed: "A3"
- board text removed: "A4"
- board text removed: "A5"
- board text removed: "A6"
- board text removed: "A7"
- board text removed: "A8"
- board text removed: "A9"
- board text removed: "D0"
- board text removed: "D1"
- board text removed: "D2"
- board text removed: "D3"
- board text removed: "D4"
- board text removed: "D5"
- board text removed: "D6"
- board text removed: "D7"
- board text removed: "GB-BRK-CART v4.0 https://gekkio.fi"
- board text removed: "GND"
- board text removed: "PHI"
- board text removed: "VIN"
- board text removed: "~{CS}"
- board text removed: "~{RD}"
- board text removed: "~{RES}"
- board text removed: "~{WR}"
