File: GB-ICECART-GB-Alpha/GB-ICECART-GB.kicad_sch (KiCad schematic)
At the start: 53 parts, among them J1 DNF, J2 TYPE-C-31-M-12, J3 AudioJack3, J4 Conn_02x08_Odd_Even, J5 Micro_SD_Card_Det, Q1 AO3401A, Q2 AO3401A, SW1 SW_Push, U1 STM32F407ZGTx, U2 HT75xx-1-SOT89, U3 IS66WVS4M8BLL-104NLI, Y1 Crystal 8M

Commit message: Preliminary routing and BOM
Parts:
- removed BT1: Battery_Cell, Battery:BatteryHolder_Keystone_3002_1x2032, symbol Device:Battery_Cell
- removed D1: D_Schottky, Diode_SMD:D_0201_0603Metric, symbol Device:D_Schottky
- removed MK2: DNF, Gekkio_MountingHole:MountingHole_2.3mm, symbol Mechanical:Mounting_Hole
- removed Q2: AO3401A, Package_TO_SOT_SMD:SOT-23, symbol Transistor_FET:AO3401A
- removed R12: 100K, Resistor_SMD:R_0603_1608Metric, symbol Device:R_US
Connections:
- net PWR_LED is gone; now on net VDD: R5.1
- net 3.3V: no longer SW1.1
- net LED1: now also U1.34 (PA0); no longer U1.1 (PE2)
- net LED2: now also U1.35 (PA1); no longer U1.2 (PE3)
- net LED3: now also U1.36 (PA2); no longer U1.3 (PE4)
- net VDD: now also SW1.1
- net at R5.2: now also LD2.2 (A); no longer LD1.2 (A)
- net at R7.2: now also LD1.2 (A); no longer LD3.2 (A)
- net at R6.2: now also LD3.2 (A); no longer LD2.2 (A)
- net VBAT: no longer names the net of C16.1, R16.2
- net VBAT: no longer U1.6 (VBAT)
- no-connect marks 3 -> 50
Other:
- note removed: "Battery"
- moved on the sheet: LD1, LD2, LD3
